File: motorized-faders/display.kicad_sch (KiCad schematic)
At the start: 1 part, among them J1 Conn_01x08

Commit message: kicad: assign all footprints
Parts:
- J1: footprint (none) -> Connector_PinHeader_2.54mm:PinHeader_1x08_P2.54mm_Vertical
Changed lines of the file:
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@@
 			)
 		)
-		(property "Footprint" ""
+		(property "Footprint" "Connector_PinHeader_2.54mm:PinHeader_1x08_P2.54mm_Vertical"
 			(at 152.4 76.2 0)
 			(hide yes)

Commit message: pcb: header wiring not soldered, add mounting holes, place components
Parts:
- renumbered J1 to J_DISP1
Changed lines of the file:
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@@
 		(dnp no)
 		(fields_autoplaced yes)
-		(property "Reference" "J1"
+		(property "Reference" "J_DISP1"
 			(at 152.4 59.69 0)
 			(show_name no)
@@
 			(project "motorized-faders"
 				(path "/b7e3fc1e-7c8d-4632-8bd7-928f8e22b8b2/0326868e-5350-4727-9104-7da40ae8c021"
-					(reference "J3")
+					(reference "J_DISP3")
 					(unit 1)
 				)
 				(path "/b7e3fc1e-7c8d-4632-8bd7-928f8e22b8b2/85403017-6d05-490d-9e30-efef74dcb89f"
-					(reference "J1")
+					(reference "J_DISP1")
 					(unit 1)
 				)
 				(path "/b7e3fc1e-7c8d-4632-8bd7-928f8e22b8b2/b1ac9845-4a2d-40da-b03b-ec1b21e58a45"
-					(reference "J6")
+					(reference "J_DISP4")
 					(unit 1)
 				)
 				(path "/b7e3fc1e-7c8d-4632-8bd7-928f8e22b8b2/d203f622-5b76-4971-ac77-8585991a3fe5"
-					(reference "J2")
+					(reference "J_DISP2")
 					(unit 1)
 				)
