File: motorized-faders/display.kicad_sch (KiCad schematic)
At the start: 1 part

Commit message: hw: single keyed JST-XH connector per fader and per display
Replace the per-fader 1x02 motor + 1x03 wiper/power headers with one
B5B-XH-A (MOTOR_A, MOTOR_B, GND, WIPER, 3V3) and move display headers to
B8B-XH-A in the same family. Keyed housings prevent reversed plugs
shorting 3.3 V to GND. PCB layout still needs Update from Schematic.

Co-Authored-By: Claude Opus 5.5 <noreply@anthropic.com>
Claude-Session: https://claude.ai/code/session_01KVW9PXPtP6oAbBUGi54MaJ
Parts:
- J_DISP1: value Conn_01x08 -> B8B-XH-A; footprint Connector_PinHeader_2.54mm:PinHeader_1x08_P2.54mm_Vertical -> Connector_JST:JST_XH_B8B-XH-A_1x08_P2.50mm_Vertical
Changed lines of the file:
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@@
 			)
 		)
-		(property "Value" "Conn_01x08"
+		(property "Value" "B8B-XH-A"
 			(at 152.4 62.23 0)
 			(show_name no)
@@
 			)
 		)
-		(property "Footprint" "Connector_PinHeader_2.54mm:PinHeader_1x08_P2.54mm_Vertical"
+		(property "Footprint" "Connector_JST:JST_XH_B8B-XH-A_1x08_P2.50mm_Vertical"
 			(at 152.4 76.2 0)
 			(hide yes)
