File: motorized-faders/fader.kicad_sch (KiCad schematic)
At the start: 2 parts, among them J4 Conn_01x03, J5 Conn_01x02

Commit message: kicad: assign all footprints
Parts:
- J4: footprint Display:CR2013-MI2120 -> Connector_PinHeader_2.54mm:PinHeader_1x03_P2.54mm_Vertical
- J5: footprint Display:CR2013-MI2120 -> Connector_PinHeader_2.54mm:PinHeader_1x02_P2.54mm_Vertical
Changed lines of the file:
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@@
 			)
 		)
-		(property "Footprint" "Display:CR2013-MI2120"
+		(property "Footprint" "Connector_PinHeader_2.54mm:PinHeader_1x02_P2.54mm_Vertical"
 			(at 184.15 58.42 0)
 			(hide yes)
@@
 			)
 		)
-		(property "Footprint" "Display:CR2013-MI2120"
+		(property "Footprint" "Connector_PinHeader_2.54mm:PinHeader_1x03_P2.54mm_Vertical"
 			(at 154.94 58.42 0)
 			(hide yes)

Commit message: pcb: header wiring not soldered, add mounting holes, place components
Parts:
- renumbered J4 to J_F1_GEN1, J5 to J_F1_MOT1
Changed lines of the file:
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@@
 		(dnp no)
 		(fields_autoplaced yes)
-		(property "Reference" "J5"
+		(property "Reference" "J_F1_MOT1"
 			(at 184.15 49.53 0)
 			(show_name no)
@@
 			(project "motorized-faders"
 				(path "/b7e3fc1e-7c8d-4632-8bd7-928f8e22b8b2/64389fec-fb00-4186-b5b1-261536e6c62d"
-					(reference "J10")
+					(reference "J_F3_MOT1")
 					(unit 1)
 				)
 				(path "/b7e3fc1e-7c8d-4632-8bd7-928f8e22b8b2/889cac32-bfc7-4106-895c-77c1ed4d1afb"
-					(reference "J8")
+					(reference "J_F2_MOT1")
 					(unit 1)
 				)
 				(path "/b7e3fc1e-7c8d-4632-8bd7-928f8e22b8b2/bac43807-ad40-4bbd-b72a-4b10a47f3691"
-					(reference "J12")
+					(reference "J_F4_MOT1")
 					(unit 1)
 				)
 				(path "/b7e3fc1e-7c8d-4632-8bd7-928f8e22b8b2/df0197ea-43aa-4e80-8ac6-816dff1fb039"
-					(reference "J5")
+					(reference "J_F1_MOT1")
 					(unit 1)
 				)
@@
 		(dnp no)
 		(fields_autoplaced yes)
-		(property "Reference" "J4"
+		(property "Reference" "J_F1_GEN1"
 			(at 154.94 49.53 0)
 			(show_name no)
@@
 			(project "motorized-faders"
 				(path "/b7e3fc1e-7c8d-4632-8bd7-928f8e22b8b2/64389fec-fb00-4186-b5b1-261536e6c62d"
-					(reference "J9")
+					(reference "J_F3_GEN1")
 					(unit 1)
 				)
 				(path "/b7e3fc1e-7c8d-4632-8bd7-928f8e22b8b2/889cac32-bfc7-4106-895c-77c1ed4d1afb"
-					(reference "J7")
+					(reference "J_F2_GEN1")
 					(unit 1)
 				)
 				(path "/b7e3fc1e-7c8d-4632-8bd7-928f8e22b8b2/bac43807-ad40-4bbd-b72a-4b10a47f3691"
-					(reference "J11")
+					(reference "J_F4_GEN1")
 					(unit 1)
 				)
 				(path "/b7e3fc1e-7c8d-4632-8bd7-928f8e22b8b2/df0197ea-43aa-4e80-8ac6-816dff1fb039"
-					(reference "J4")
+					(reference "J_F1_GEN1")
 					(unit 1)
 				)
