File: motorized-faders/motorized-faders.kicad_pcb (KiCad board)
At the start: 2 copper layers, 131 x 93 mm, 62 parts

Commit message: pcb: route signal and power traces, grounds pending
Parts:
- moved J_DISP4 110.3 mm to (66.9, 53.5), turned to 90 degrees
- moved U_MOT_B1 102.7 mm to (169.0, 67.5), turned to 180 degrees
- moved C_VM_B1 96.7 mm to (159.5, 74.0), turned to 90 degrees
- moved C_VCC_B1 95.8 mm to (168.0, 58.5), turned to 90 degrees
- moved J_DISP3 95.7 mm to (66.8, 68.5), turned to 90 degrees
- moved C_VM_B_HF1 91.6 mm to (162.5, 63.0), turned to 90 degrees
- moved R_DISP_RES1 88.8 mm to (59.8, 91.0), turned to 90 degrees
- moved TP_GND2 86.0 mm to (158.5, 62.0), turned to 90 degrees
- moved C_DISP_RES1 85.9 mm to (59.8, 98.5), turned to 90 degrees
- moved J_DISP2 83.9 mm to (66.8, 83.5), turned to 90 degrees
- moved J_DISP1 76.3 mm to (66.8, 98.5), turned to 90 degrees
- moved U_MOT_A1 75.1 mm to (145.0, 67.5), turned to 180 degrees
- moved C_VM_A1 73.1 mm to (135.5, 74.0), turned to 90 degrees
- moved C_VCC_A1 66.0 mm to (144.0, 58.5), turned to 90 degrees
- moved TP_SCK1 64.9 mm to (69.5, 49.3)
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Routing:
- net +3V3: track 0.00 -> 238.4 mm, vias 0 -> 4
- net /SPI_MOSI: track 0.00 -> 136.7 mm, vias 0 -> 1
- net /F4_WIPER: track 0.00 -> 125.2 mm
- net /SPI_SCK: track 0.00 -> 122.5 mm, vias 0 -> 2
- net /BTN_GEN: track 0.00 -> 109.2 mm
- net /F3_WIPER: track 0.00 -> 105.7 mm
- net /DISP_RES: track 0.00 -> 103.0 mm
- net /DISP_DC: track 0.00 -> 95.2 mm
- net /B_PWMB: track 0.00 -> 89.0 mm, vias 0 -> 1
- net /B_BIN2: track 0.00 -> 88.1 mm, vias 0 -> 1
- net /F2_WIPER: track 0.00 -> 86.5 mm, vias 0 -> 1
- net /B_BIN1: track 0.00 -> 83.3 mm, vias 0 -> 1
- net /B_AIN2: track 0.00 -> 80.5 mm, vias 0 -> 1
- net /B_AIN1: track 0.00 -> 80.3 mm, vias 0 -> 1
- net /B_PWMA: track 0.00 -> 79.7 mm, vias 0 -> 1
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
Commit message: pcb: grounds, first DRC errors fixed
Routing:
- net GND: track 4.00 -> 147.2 mm, vias 0 -> 15
- net +3V3: track 238.4 -> 352.7 mm, vias 4 -> 6
- net +9V: track 78.3 -> 168.4 mm, vias 0 -> 4
- net GNDPWR: track 53.6 -> 65.6 mm, vias 0 -> 3
- net /STBY: track 63.0 -> 66.3 mm
- net /DISP1_CS: track 42.3 -> 43.2 mm
- added copper zone on B.Cu, net GND
- added copper zone on B.Cu, net GNDPWR

Commit message: pcb: add TB6612 breakout headers, finish routing and grounds
Parts:
- added J_MOT_BOB_A_P1: Conn_01x08, Connector_PinHeader_2.54mm:PinHeader_1x08_P2.54mm_Vertical, F.Cu at (204.6, 57.6)
- added J_MOT_BOB_A_P2: Conn_01x08, Connector_PinHeader_2.54mm:PinHeader_1x08_P2.54mm_Vertical, F.Cu at (204.6, 75.4)
- added J_MOT_BOB_B_P1: Conn_01x08, Connector_PinHeader_2.54mm:PinHeader_1x08_P2.54mm_Vertical, F.Cu at (204.6, 84.9)
- added J_MOT_BOB_B_P2: Conn_01x08, Connector_PinHeader_2.54mm:PinHeader_1x08_P2.54mm_Vertical, F.Cu at (204.6, 102.7)
- REF** (x4): value MountingHole_3.2mm_M3 -> 3.2mm M3
- moved REF** 24.0 mm to (205.0, 48.0)
- moved REF** 24.0 mm to (205.0, 131.0)
- renumbered C_BTN_FADER1 to C_BTN_FADER, C_BTN_GEN1 to C_BTN_GEN, C_DISP_RES1 to C_DISP_RES, C_F1_WIPER1 to C_F1_WIPER, C_F2_WIPER1 to C_F2_WIPER, C_F3_WIPER1 to C_F3_WIPER, C_F4_WIPER1 to C_F4_WIPER, C_MCP3208_VDD_GND1 to C_MCP3208_VDD_GND, C_MCP3208_VREF_GND1 to C_MCP3208_VREF_GND, C_VCC_A1 to C_VCC_A, C_VCC_B1 to C_VCC_B, C_VM_A1 to C_VM_A, C_VM_A_HF1 to C_VM_A_HF, C_VM_B1 to C_VM_B, C_VM_B_HF1 to C_VM_B_HF, J_PD1 to J_PD, R_BTN_FADER1 to R_BTN_FADER, R_BTN_GEN_PU1 to R_BTN_GEN, R_DISP_RES1 to R_DISP_RES, R_F1_WIPER1 to R_F1_WIPER, R_F2_WIPER1 to R_F2_WIPER, R_F3_WIPER1 to R_F3_WIPER, R_F4_WIPER1 to R_F4_WIPER, R_VM_SENSE_BOT1 to R_VM_SENSE_BOT, R_VM_SENSE_TOP1 to R_VM_SENSE_TOP, TP_F1_ADC1 to TP_F1_ADC, TP_GND1 to TP_GND, TP_GND2 to TP_GNDPWR, TP_SCK1 to TP_SCK, U_ADC1 to U_ADC, U_MOT_A1 to U_MOT_A, U_MOT_B1 to U_MOT_B
Routing:
- net /A_BIN1: track 56.7 -> 175.9 mm, vias 1 -> 2
- net /A_BIN2: track 53.5 -> 172.3 mm, vias 2 -> 3
- net +9V: track 168.4 -> 282.5 mm
- net /A_PWMB: track 54.3 -> 162.1 mm, vias 1 -> 2
- net /A_AIN1: track 55.0 -> 160.1 mm, vias 1 -> 3
- net /A_AIN2: track 53.2 -> 154.2 mm, vias 1 -> 3
- net /A_PWMA: track 53.8 -> 147.3 mm
- net /F1_MOT_A: track 28.7 -> 119.0 mm
- net +3V3: track 352.7 -> 441.7 mm, vias 6 -> 7
- net /F1_MOT_B: track 29.2 -> 118.1 mm
- net /F2_MOT_A: track 29.5 -> 100.6 mm
- net /B_PWMB: track 89.0 -> 157.3 mm, vias 1 -> 3
- net /STBY: track 66.3 -> 134.2 mm, vias 3 -> 5
- net /B_BIN2: track 88.1 -> 153.7 mm, vias 1 -> 3
- net /B_BIN1: track 83.3 -> 146.3 mm, vias 1 -> 3
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Other:
- board size 131 x 93 mm -> 155 x 93 mm
